Commit message: init analyze

File: body.urdf (robot description, URDF)
Before this commit: robot robot, 3 links, 2 joints
Links:
- removed link back_leg
- removed link front_leg
- removed link torso
- added link BackLeg, mass 1; collision box size=1 1 1; visual box size=1 1 1
- added link FrontLeg, mass 1; collision box size=1 1 1; visual box size=1 1 1
- added link Torso, mass 1; collision box size=1 1 1; visual box size=1 1 1
Joints:
- removed joint Torso_Leg
- removed joint Torso_Leg2
- added joint Torso_BackLeg: type revolute, parent Torso, child BackLeg, origin xyz=1 0 1 rpy=0 0 0, axis 0 1 0, limit lower=-3.14159 upper=3.14159 effort=0.0 velocity=0.0
- added joint Torso_FrontLeg: type revolute, parent Torso, child FrontLeg, origin xyz=2 0 1 rpy=0 0 0, axis 0 1 0, limit lower=-3.14159 upper=3.14159 effort=0.0 velocity=0.0

Commit message: push

File: body.urdf (robot description, URDF)
Before this commit: robot robot, 3 links, 2 joints
Links:
- added link BackLegBottom, mass 1; collision box size=0.2 0.2 1; visual box size=0.2 0.2 1
- added link FrontLegBottom, mass 1; collision box size=0.2 0.2 1; visual box size=0.2 0.2 1
- added link LeftLeg, mass 1; collision box size=1 0.2 0.2; visual box size=1 0.2 0.2
- added link LeftLegBottom, mass 1; collision box size=0.2 0.2 1; visual box size=0.2 0.2 1
- added link RightLeg, mass 1; collision box size=1 0.2 0.2; visual box size=1 0.2 0.2
- added link RightLegBottom, mass 1; collision box size=0.2 0.2 1; visual box size=0.2 0.2 1
- link BackLeg: geometry collision box size=0.2 1 0.2; visual box size=0.2 1 0.2
- link FrontLeg: geometry collision box size=0.2 1 0.2; visual box size=0.2 1 0.2
Joints:
- added joint BackLeg_BackLegBottom: type revolute, parent BackLeg, child BackLegBottom, origin xyz=0 -1 0 rpy=0 0 0, axis 1 0 0, limit lower=-3.14159 upper=3.14159 effort=0.0 velocity=0.0
- added joint FrontLeg_FrontLegBottom: type revolute, parent FrontLeg, child FrontLegBottom, origin xyz=0 1 0 rpy=0 0 0, axis 1 0 0, limit lower=-3.14159 upper=3.14159 effort=0.0 velocity=0.0
- added joint LeftLeg_LeftLegBottom: type revolute, parent LeftLeg, child LeftLegBottom, origin xyz=1 0 0 rpy=0 0 0, axis 0 1 0, limit lower=-3.14159 upper=3.14159 effort=0.0 velocity=0.0
- added joint RightLeg_RightLegBottom: type revolute, parent RightLeg, child RightLegBottom, origin xyz=-1 0 0 rpy=0 0 0, axis 0 1 0, limit lower=-3.14159 upper=3.14159 effort=0.0 velocity=0.0
- added joint Torso_LeftLeg: type revolute, parent Torso, child LeftLeg, origin xyz=0.5 0 1 rpy=0 0 0, axis 0 1 0, limit lower=-3.14159 upper=3.14159 effort=0.0 velocity=0.0
- added joint Torso_RightLeg: type revolute, parent Torso, child RightLeg, origin xyz=-0.5 0 1 rpy=0 0 0, axis 0 1 0, limit lower=-3.14159 upper=3.14159 effort=0.0 velocity=0.0
- joint Torso_BackLeg: axis 0 1 0 -> 1 0 0; origin xyz=1 0 1 rpy=0 0 0 -> xyz=0 -0.5 1 rpy=0 0 0
- joint Torso_FrontLeg: axis 0 1 0 -> 1 0 0; origin xyz=2 0 1 rpy=0 0 0 -> xyz=0 0.5 1 rpy=0 0 0

Commit message: added some legs

File: body.urdf (robot description, URDF)
Before this commit: robot robot, 9 links, 8 joints
Links:
- added link BackLeg2, mass 1; collision box size=0.2 1 0.2; visual box size=0.2 1 0.2
- added link BackLegBottom2, mass 1; collision box size=0.2 0.2 1; visual box size=0.2 0.2 1
- added link FrontLeg2, mass 1; collision box size=0.2 1 0.2; visual box size=0.2 1 0.2
- added link FrontLegBottom2, mass 1; collision box size=0.2 0.2 1; visual box size=0.2 0.2 1
Joints:
- added joint BackLeg_BackLegBottom2: type revolute, parent BackLeg2, child BackLegBottom2, origin xyz=0 -1 0 rpy=0 0 0, axis 1 0 0, limit lower=-3.14159 upper=3.14159 effort=0.0 velocity=0.0
- added joint FrontLeg_FrontLegBottom2: type revolute, parent FrontLeg2, child FrontLegBottom2, origin xyz=0 1 0 rpy=0 0 0, axis 1 0 0, limit lower=-3.14159 upper=3.14159 effort=0.0 velocity=0.0
- added joint Torso_BackLeg2: type revolute, parent Torso, child BackLeg2, origin xyz=0 -0.5 1 rpy=0 0 0, axis 1 0 0, limit lower=-3.14159 upper=3.14159 effort=0.0 velocity=0.0
- added joint Torso_FrontLeg2: type revolute, parent Torso, child FrontLeg2, origin xyz=0 0.5 1 rpy=0 0 0, axis 1 0 0, limit lower=-3.14159 upper=3.14159 effort=0.0 velocity=0.0

Commit message: scorpion

File: body.urdf (robot description, URDF)
Before this commit: robot robot, 13 links, 12 joints
Links:
- removed link LeftLeg
- removed link LeftLegBottom
- added link BackLeg3, mass 1; collision box size=0.2 1 0.2; visual box size=0.2 1 0.2
- added link BackLegBottom3, mass 1; collision box size=0.1 0.1 1; visual box size=0.1 0.1 1
- added link FrontLeg3, mass 1; collision box size=0.2 1 0.2; visual box size=0.2 1 0.2
- added link FrontLegBottom3, mass 1; collision box size=0.1 0.1 1; visual box size=0.1 0.1 1
Joints:
- removed joint LeftLeg_LeftLegBottom
- removed joint Torso_LeftLeg
- added joint BackLeg_BackLegBottom3: type revolute, parent BackLeg3, child BackLegBottom3, origin xyz=0 -1 0 rpy=0 0 0, axis 1 0 0, limit lower=-3.14159 upper=3.14159 effort=0.0 velocity=0.0
- added joint FrontLeg_FrontLegBottom3: type revolute, parent FrontLeg3, child FrontLegBottom3, origin xyz=0 1 0 rpy=0 0 0, axis 1 0 0, limit lower=-3.14159 upper=3.14159 effort=0.0 velocity=0.0
- added joint Torso_BackLeg3: type revolute, parent Torso, child BackLeg3, origin xyz=0 -0.5 1 rpy=0 0 0, axis 1 0 0, limit lower=-3.14159 upper=3.14159 effort=0.0 velocity=0.0
- added joint Torso_FrontLeg3: type revolute, parent Torso, child FrontLeg3, origin xyz=0 0.5 1 rpy=0 0 0, axis 1 0 0, limit lower=-3.14159 upper=3.14159 effort=0.0 velocity=0.0

Commit message: working

File: body.urdf (robot description, URDF)
Before this commit: robot robot, 15 links, 14 joints
Links:
- removed link BackLeg
- removed link BackLeg2
- removed link BackLeg3
- removed link BackLegBottom
- removed link BackLegBottom2
- removed link BackLegBottom3
- removed link FrontLeg
- removed link FrontLeg2
- removed link FrontLeg3
- removed link FrontLegBottom
- removed link FrontLegBottom2
- removed link FrontLegBottom3
- removed link RightLeg
- removed link RightLegBottom
- removed link Torso
- added link Head, mass 1; collision box size=0.3421407371440314 0.17220456429161485 0.6368261315858854; visual box size=0.3421407371440314 0.17220456429161485 0.6368261315858854
- added link b0, mass 1; collision box size=0.6621200821097591 0.9443879767576437 1.0050160900774379; visual box size=0.6621200821097591 0.9443879767576437 1.0050160900774379
- added link b1, mass 1; collision box size=0.09234140030676426 0.8543963691212506 0.5398709201067863; visual box size=0.09234140030676426 0.8543963691212506 0.5398709201067863
- added link b2, mass 1; collision box size=1.0481023239233298 0.5161604438136451 0.6028913167039596; visual box size=1.0481023239233298 0.5161604438136451 0.6028913167039596
- added link b3, mass 1; collision box size=0.7695193699538131 0.3186852624142151 0.21376669994244496; visual box size=0.7695193699538131 0.3186852624142151 0.21376669994244496
- added link b4, mass 1; collision box size=0.18222479552472154 0.20308188440334468 0.4302999136272612; visual box size=0.18222479552472154 0.20308188440334468 0.4302999136272612
Joints:
- removed joint BackLeg_BackLegBottom
- removed joint BackLeg_BackLegBottom2
- removed joint BackLeg_BackLegBottom3
- removed joint FrontLeg_FrontLegBottom
- removed joint FrontLeg_FrontLegBottom2
- removed joint FrontLeg_FrontLegBottom3
- removed joint RightLeg_RightLegBottom
- removed joint Torso_BackLeg
- removed joint Torso_BackLeg2
- removed joint Torso_BackLeg3
- removed joint Torso_FrontLeg
- removed joint Torso_FrontLeg2
- removed joint Torso_FrontLeg3
- removed joint Torso_RightLeg
- added joint j_0: type revolute, parent Head, child b0, origin xyz=0 0.08610228214580742 0.5 rpy=0 0 0, axis 1 0 0, limit lower=-3.14159 upper=3.14159 effort=0.0 velocity=0.0
- added joint j_1: type revolute, parent b0, child b1, origin xyz=0 0.08610228214580742 0 rpy=0 0 0, axis 1 0 0, limit lower=-3.14159 upper=3.14159 effort=0.0 velocity=0.0
- added joint j_2: type revolute, parent b1, child b2, origin xyz=0 0.08610228214580742 0 rpy=0 0 0, axis 1 0 0, limit lower=-3.14159 upper=3.14159 effort=0.0 velocity=0.0
- added joint j_3: type revolute, parent b2, child b3, origin xyz=0 0.08610228214580742 0 rpy=0 0 0, axis 1 0 0, limit lower=-3.14159 upper=3.14159 effort=0.0 velocity=0.0
- added joint j_4: type revolute, parent b3, child b4, origin xyz=0 0.08610228214580742 0 rpy=0 0 0, axis 1 0 0, limit lower=-3.14159 upper=3.14159 effort=0.0 velocity=0.0

Commit message: diagram

File: body.urdf (robot description, URDF)
Before this commit: robot robot, 8 links, 7 joints
Links:
- removed link Block3
- removed link Block4
- removed link Block5
- removed link Block6
- link Block0: geometry collision box size=0.9443870964647999 0.2185945800835336 0.3589829335575604; visual box size=0.9443870964647999 0.2185945800835336 0.3589829335575604
- link Block1: geometry collision box size=0.7644985603397131 0.6343073319125575 0.8109758100493487; visual box size=0.7644985603397131 0.6343073319125575 0.8109758100493487
- link Block2: geometry collision box size=0.5255787762048557 0.12053362501708774 0.5238504840173076; visual box size=0.5255787762048557 0.12053362501708774 0.5238504840173076
- link Torso: geometry collision box size=0.8975600743097087 0.8932508297276442 0.17077659219122898; visual box size=0.8975600743097087 0.8932508297276442 0.17077659219122898
Joints:
- removed joint Block2_Block3
- removed joint Block3_Block4
- removed joint Block4_Block5
- removed joint Block5_Block6

Commit message: cleaned up

File: body.urdf (robot description, URDF)
Before this commit: robot robot, 4 links, 3 joints
Links:
- added link Block3, mass 1; collision box size=0.3631341466317317 0.05188567572749191 0.7532985114153139; visual box size=0.3631341466317317 0.05188567572749191 0.7532985114153139
- link Block0: geometry collision box size=0.3593695612884613 0.07897675253252755 0.7255903647976434; visual box size=0.3593695612884613 0.07897675253252755 0.7255903647976434
- link Block1: geometry collision box size=0.3460631925009927 0.277594738079443 0.7254891466703048; visual box size=0.3460631925009927 0.277594738079443 0.7254891466703048
- link Block2: geometry collision box size=0.4561867395645859 1.580638566481863 0.7984699482394035; visual box size=0.4561867395645859 1.580638566481863 0.7984699482394035
- link Torso: geometry collision box size=0.7064415333370083 0.6349178984076185 0.4361852952288675; visual box size=0.7064415333370083 0.6349178984076185 0.4361852952288675
Joints:
- added joint Block2_Block3: type revolute, parent Block2, child Block3, origin xyz=0.22809336978229294 0.7903192832409315 0 rpy=0 0 0, axis 1 0 0, limit lower=-3.14159 upper=3.14159 effort=0.0 velocity=0.0
- joint Block0_Block1: origin xyz=0 0.0 0 rpy=0 0 0 -> xyz=0.17968478064423066 0.039488376266263774 0 rpy=0 0 0
- joint Block1_Block2: origin xyz=0 0.0 0 rpy=0 0 0 -> xyz=0 0.1387973690397215 0 rpy=0 0 0
- joint Torso_Block0: origin xyz=0 0 0.5 rpy=0 0 0 -> xyz=0.35322076666850416 0 0.5 rpy=0 0 0
